Commit message: Update the model for LAAS-CNRS robot with camera by default.

File: robots/common/franka_arm.xacro (robot description, xacro)
@@ -5,5 +5,5 @@
   <!-- arm_id: Namespace of the robot arm. Serves to differentiate between arms in case of multiple instances. -->
   <!-- joint_limits: description of the joint limits that comes from a YAML file. Example definition: ${xacro.load_yaml('$(find franka_description)/robots/fr3/joint_limits.yaml')} -->
-  <xacro:macro name="franka_arm" params="arm_id:='panda' description_pkg:='franka_description' connected_to:='' xyz:='0 0 0' rpy:='0 0 0' gazebo:=false safety_distance:=0 joint_limits" >
+  <xacro:macro name="franka_arm" params="arm_id:='panda' description_pkg:='franka_description' connected_to:='' xyz:='0 0 0' rpy:='0 0 0' self_col:=false safety_distance:=0 joint_limits" >
     <xacro:unless value="${not connected_to}">
       <joint name="${arm_id}_joint_${connected_to}" type="fixed">
@@ -13,10 +13,10 @@
       </joint>
     </xacro:unless>
-    <xacro:link_with_sc name="link0" gazebo="${gazebo}">
+    <xacro:link_with_sc name="link0" self_col="${self_col}">
       <self_collision_geometries>
         <xacro:collision_capsule xyz="-0.075 0 0.06" direction="x" radius="${0.06+safety_distance}" length="0.03" />
       </self_collision_geometries>
     </xacro:link_with_sc>
-    <xacro:link_with_sc name="link1" gazebo="${gazebo}">
+    <xacro:link_with_sc name="link1" self_col="${self_col}">
       <self_collision_geometries>
         <xacro:collision_capsule xyz="0 0 -191.5e-3" radius="${0.06+safety_distance}" length="0.283" />
@@ -31,5 +31,5 @@
       <dynamics D="1" K="7000" damping="0.003" friction="0.0" mu_coulomb="0" mu_viscous="16" />
     </joint>
-    <xacro:link_with_sc name="link2" gazebo="${gazebo}">
+    <xacro:link_with_sc name="link2" self_col="${self_col}">
       <self_collision_geometries>
         <xacro:collision_capsule xyz="0 0 0" radius="${0.06+safety_distance}" length="0.12" />
@@ -44,5 +44,5 @@
       <dynamics D="1" K="7000" damping="0.003" friction="0.0" mu_coulomb="0" mu_viscous="16" />
     </joint>
-    <xacro:link_with_sc name="link3" gazebo="${gazebo}">
+    <xacro:link_with_sc name="link3" self_col="${self_col}">
       <self_collision_geometries>
         <xacro:collision_capsule xyz="0 0 -0.145" radius="${0.06+safety_distance}" length="0.15" />
@@ -57,5 +57,5 @@
       <dynamics D="1" K="7000" damping="0.003" friction="0.0" mu_coulomb="0" mu_viscous="16" />
     </joint>
-    <xacro:link_with_sc name="link4" gazebo="${gazebo}">
+    <xacro:link_with_sc name="link4" self_col="${self_col}">
       <self_collision_geometries>
         <xacro:collision_capsule xyz="0 0 0" radius="${0.06+safety_distance}" length="0.12" />
@@ -70,5 +70,5 @@
       <dynamics D="1" K="7000" damping="0.003" friction="0.0" mu_coulomb="0" mu_viscous="16" />
     </joint>
-    <xacro:link_with_sc name="link5" gazebo="${gazebo}">
+    <xacro:link_with_sc name="link5" self_col="${self_col}">
       <self_collision_geometries>
         <xacro:collision_capsule xyz="0 0 -0.26"    radius="${0.060+safety_distance}" length="0.10" />
@@ -84,5 +84,5 @@
       <dynamics D="1" K="7000" damping="0.003" friction="0.0" mu_coulomb="0" mu_viscous="16" />
     </joint>
-    <xacro:link_with_sc name="link6" gazebo="${gazebo}">
+    <xacro:link_with_sc name="link6" self_col="${self_col}">
       <self_collision_geometries>
         <xacro:collision_capsule xyz="0 0 -0.03" radius="${0.05+safety_distance}" length="0.08" />
@@ -97,5 +97,5 @@
       <dynamics D="1" K="7000" damping="0.003" friction="0.0" mu_coulomb="0" mu_viscous="16" />
     </joint>
-    <xacro:link_with_sc name="link7" gazebo="${gazebo}" rpy="0 0 ${pi/4}">
+    <xacro:link_with_sc name="link7" self_col="${self_col}" rpy="0 0 ${pi/4}">
       <self_collision_geometries>
         <xacro:collision_capsule xyz="0 0 0.01" direction="z" radius="${0.04+safety_distance}" length="0.14" />
@@ -111,5 +111,7 @@
       <dynamics D="1" K="7000" damping="0.003" friction="0.0" mu_coulomb="0" mu_viscous="16"/>
     </joint>
-    <link name="${arm_id}_link8"/>
+    <link name="${arm_id}_link8">
+      <xacro:inertial_props name="zero_inertia"/>
+    </link>
     <joint name="${arm_id}_joint8" type="fixed">
       <origin rpy="0 0 0" xyz="0 0 0.107"/>

File: robots/common/franka_hand.xacro (robot description, xacro)
@@ -2,5 +2,5 @@
 <robot xmlns:xacro="http://www.ros.org/wiki/xacro" name="hand">
   <!-- safety_distance: Minimum safety distance in [m] by which the collision volumes are expanded and which is enforced during robot motions -->
-  <xacro:macro name="franka_hand" params="connected_to:='' arm_id:='panda' rpy:='0 0 0' xyz:='0 0 0' tcp_xyz:='0 0 0.1034' tcp_rpy:='0 0 0' safety_distance:=0 gazebo:=false description_pkg:=franka_description">
+  <xacro:macro name="franka_hand" params="connected_to:='' arm_id:='panda' rpy:='0 0 0' xyz:='0 0 0' tcp_xyz:='0 0 0.1034' tcp_rpy:='0 0 0' safety_distance:=0 self_col:=false description_pkg:=franka_description hand_col:=false convex_col:=false">
     <xacro:unless value="${connected_to == ''}">
       <joint name="${arm_id}_hand_joint" type="fixed">
@@ -10,12 +10,14 @@
       </joint>
     </xacro:unless>
-    <xacro:link_with_sc name="hand" gazebo="${gazebo}">
+    <xacro:link_with_sc name="hand" self_col="${hand_col}">
       <self_collision_geometries>
-        <xacro:collision_capsule xyz="0 0 0.04" direction="y" radius="${0.04+safety_distance}" length="0.1" />
-        <xacro:collision_capsule xyz="0 0 0.10" direction="y" radius="${0.02+safety_distance}" length="0.1" />
+          <xacro:collision_capsule xyz="0 0 0.04" direction="y" radius="${0.04+safety_distance}" length="0.1" />
+          <xacro:collision_capsule xyz="0 0 0.10" direction="y" radius="${0.02+safety_distance}" length="0.1" />
       </self_collision_geometries>
     </xacro:link_with_sc>
     <!-- Define the hand_tcp frame -->
-    <link name="${arm_id}_hand_tcp" />
+    <link name="${arm_id}_hand_tcp">
+      <xacro:inertial_props name="zero_inertia"/>
+    </link>
     <joint name="${arm_id}_hand_tcp_joint" type="fixed">
       <origin xyz="${tcp_xyz}" rpy="${tcp_rpy}" />
@@ -29,35 +31,44 @@
         </geometry>
       </visual>
-      <!-- screw mount -->
-      <collision>
-        <origin xyz="0 18.5e-3 11e-3" rpy="0 0 0" />
-        <geometry>
-          <box size="22e-3 15e-3 20e-3" />
-        </geometry>
-      </collision>
-      <!-- cartriage sledge -->
-      <collision>
-        <origin xyz="0 6.8e-3 2.2e-3" rpy="0 0 0" />
-        <geometry>
-          <box size="22e-3 8.8e-3 3.8e-3" />
-        </geometry>
-      </collision>
-      <!-- diagonal finger -->
-      <collision>
-        <origin xyz="0 15.9e-3 28.35e-3" rpy="${pi/6} 0 0" />
-        <geometry>
-          <box size="17.5e-3 7e-3 23.5e-3" />
-        </geometry>
-      </collision>
-      <!-- rubber tip with which to grasp -->
-      <collision>
-        <origin xyz="0 7.58e-3 45.25e-3" rpy="0 0 0" />
-        <geometry>
-          <box size="17.5e-3 15.2e-3 18.5e-3" />
-        </geometry>
-      </collision>
-      <xacro:if value="${gazebo}">
-        <xacro:inertial_props name="leftfinger" />
+      <xacro:if value="${convex_col}">
+        <!-- screw mount -->
+        <collision>
+          <origin rpy="0 0 0" xyz="0 18.5e-3 11e-3"/>
+          <geometry>
+            <sphere radius="0.03"/>
+          </geometry>
+        </collision>
       </xacro:if>
+      <xacro:unless value="${convex_col}">
+        <!-- screw mount -->
+        <collision>
+          <origin xyz="0 18.5e-3 11e-3" rpy="0 0 0" />
+          <geometry>
+            <box size="22e-3 15e-3 20e-3" />
+          </geometry>
+        </collision>
+        <!-- cartriage sledge -->
+        <collision>
+          <origin xyz="0 6.8e-3 2.2e-3" rpy="0 0 0" />
+          <geometry>
+            <box size="22e-3 8.8e-3 3.8e-3" />
+          </geometry>
+        </collision>
+        <!-- diagonal finger -->
+        <collision>
+          <origin xyz="0 15.9e-3 28.35e-3" rpy="${pi/6} 0 0" />
+          <geometry>
+            <box size="17.5e-3 7e-3 23.5e-3" />
+          </geometry>
+        </collision>
+        <!-- rubber tip with which to grasp -->
+        <collision>
+          <origin xyz="0 7.58e-3 45.25e-3" rpy="0 0 0" />
+          <geometry>
+            <box size="17.5e-3 15.2e-3 18.5e-3" />
+          </geometry>
+        </collision>
+      </xacro:unless>
+    <xacro:inertial_props name="leftfinger" />
     </link>
     <link name="${arm_id}_rightfinger">
@@ -68,35 +79,44 @@
         </geometry>
       </visual>
-      <!-- screw mount -->
-      <collision>
-        <origin xyz="0 -18.5e-3 11e-3" rpy="0 0 0" />
-        <geometry>
-          <box size="22e-3 15e-3 20e-3" />
-        </geometry>
-      </collision>
-      <!-- cartriage sledge -->
-      <collision>
-        <origin xyz="0 -6.8e-3 2.2e-3" rpy="0 0 0" />
-        <geometry>
-          <box size="22e-3 8.8e-3 3.8e-3" />
-        </geometry>
-      </collision>
-      <!-- diagonal finger -->
-      <collision>
-        <origin xyz="0 -15.9e-3 28.35e-3" rpy="${-pi/6} 0 0" />
-        <geometry>
-          <box size="17.5e-3 7e-3 23.5e-3" />
-        </geometry>
-      </collision>
-      <!-- rubber tip with which to grasp -->
-      <collision>
-        <origin xyz="0 -7.58e-3 45.25e-3" rpy="0 0 0" />
-        <geometry>
-          <box size="17.5e-3 15.2e-3 18.5e-3" />
-        </geometry>
-      </collision>
-      <xacro:if value="${gazebo}">
-        <xacro:inertial_props name="rightfinger" />
+      <xacro:if value="${convex_col}">
+        <!-- screw mount -->
+        <collision>
+          <origin rpy="0 0 0" xyz="0 -18.5e-3 11e-3"/>
+          <geometry>
+            <sphere radius=".03"/>
+          </geometry>
+        </collision>
       </xacro:if>
+      <xacro:unless value="${convex_col}">
+        <!-- screw mount -->
+        <collision>
+          <origin xyz="0 -18.5e-3 11e-3" rpy="0 0 0" />
+          <geometry>
+            <box size="22e-3 15e-3 20e-3" />
+          </geometry>
+        </collision>
+        <!-- cartriage sledge -->
+        <collision>
+          <origin xyz="0 -6.8e-3 2.2e-3" rpy="0 0 0" />
+          <geometry>
+            <box size="22e-3 8.8e-3 3.8e-3" />
+          </geometry>
+        </collision>
+        <!-- diagonal finger -->
+        <collision>
+          <origin xyz="0 -15.9e-3 28.35e-3" rpy="${-pi/6} 0 0" />
+          <geometry>
+            <box size="17.5e-3 7e-3 23.5e-3" />
+          </geometry>
+        </collision>
+        <!-- rubber tip with which to grasp -->
+        <collision>
+          <origin xyz="0 -7.58e-3 45.25e-3" rpy="0 0 0" />
+          <geometry>
+            <box size="17.5e-3 15.2e-3 18.5e-3" />
+          </geometry>
+        </collision>
+      </xacro:unless>
+      <xacro:inertial_props name="rightfinger" />
     </link>
     <joint name="${arm_id}_finger_joint1" type="prismatic">

File: robots/common/franka_robot.xacro (robot description, xacro)
@@ -1,8 +1,8 @@
 <?xml version='1.0' encoding='utf-8'?>
 <robot xmlns:xacro="http://www.ros.org/wiki/xacro">
-  <xacro:macro name="franka_robot" params="arm_id joint_limits parent:='world' xyz:='0 0 0' rpy:='0 0 0' hand:=false gazebo:=false tcp_xyz:='0 0 0.1034' tcp_rpy='0 0 0'">
+  <xacro:macro name="franka_robot" params="arm_id joint_limits parent:='world' xyz:='0 0 0' rpy:='0 0 0' hand:=false camera_hand:=false gazebo:=false self_col:=true hand_col:=false tcp_xyz:='0 0 0.1034' tcp_rpy:='0 0 0' convex_col:=false">
     <xacro:include filename="$(find franka_description)/robots/common/utils.xacro" />
     <xacro:include filename="$(find franka_description)/robots/common/franka_arm.xacro" />
-    <xacro:franka_arm arm_id="${arm_id}" safety_distance="0.03" gazebo="${gazebo}" joint_limits="${joint_limits}"/>
+    <xacro:franka_arm arm_id="${arm_id}" safety_distance="0.03" self_col="${self_col}" joint_limits="${joint_limits}"/>
     <xacro:if value="${hand}">
       <xacro:include filename="$(find franka_description)/robots/common/franka_hand.xacro"/>
@@ -14,6 +14,17 @@
           connected_to="${arm_id}_link8"
           safety_distance="0.03"
-          gazebo="${gazebo}"
+          self_col="${self_col}"
+          hand_col="${hand_col}"
+          convex_col="${convex_col}"
        />
+       <xacro:if value="${camera_hand}">
+        <xacro:include filename="$(find franka_description)/robots/common/camera.xacro"/>
+        <xacro:camera_hand
+            arm_id="${arm_id}"
+            rpy="0.022100209841200636 -1.3156624527412932 3.061881150974905"
+            xyz="0.13682768843416482 -0.009443400298528096 -0.08387833599341328"
+            connected_to="panda_hand"
+        />
+       </xacro:if>
     </xacro:if>
     <!-- Define additional Gazebo tags -->

File: robots/common/utils.xacro (robot description, xacro)
@@ -33,5 +33,5 @@
   <!-- self_collision_geometries:  self <collision> models        -->
   <!-- ========================================================== -->
-  <xacro:macro name="link_with_sc" params="name prefix=${arm_id}_ rpy:='0 0 0' **self_collision_geometries gazebo:=false">
+  <xacro:macro name="link_with_sc" params="name prefix=${arm_id}_ rpy:='0 0 0' self_col:=false **self_collision_geometries">
     <!-- sub-link defining detailed meshes for collision with environment -->
     <link name="${prefix}${name}">
@@ -46,13 +46,11 @@
         </geometry>
       </collision>
-      <xacro:if value="${gazebo}">
-        <xacro:inertial_props name="${name}" />
-      </xacro:if>
+      <xacro:inertial_props name="${name}" />
     </link>
     <!-- sub-link defining coarse geometries of real robot's internal self-collision -->
     <link name="${prefix}${name}_sc">
-      <xacro:unless value="${gazebo}">
+      <xacro:if value="${self_col}">
         <xacro:insert_block name="self_collision_geometries" />
-      </xacro:unless>
+      </xacro:if>
     </link>
     <!-- fixed joint between both sub-links -->

File: robots/panda/panda.urdf.xacro (robot description, xacro)
@@ -5,5 +5,11 @@
   <xacro:arg name="arm_id" default="panda" />
   <!-- Should a franka_gripper be mounted at the flange?" -->
-  <xacro:arg name="hand" default="false" />
+  <xacro:arg name="hand" default="true" />
+  <!-- Should a camera be mounted on the franka_gripper?" -->
+  <xacro:arg name="camera_hand" default="true" />
+  <!-- Should a franka_gripper use it's capsule collision?" -->
+  <xacro:arg name="hand_col" default="false" />
+  <!-- Should we use convex collision meshes?" -->
+  <xacro:arg name="convex_col" default="true" />
   <!-- Positional offset between $(arm_id)_hand -> $(arm_id)_hand_tcp [m]. Only used when hand:=true -->
   <xacro:arg name="tcp_xyz" default="0 0 0.1034" />
@@ -26,5 +32,8 @@
                       parent="$(arg parent)"
                       xyz="$(arg xyz)"
-                      rpy="$(arg rpy)">
+                      rpy="$(arg rpy)"
+                      hand_col="$(arg hand_col)"
+                      convex_col="$(arg convex_col)"
+                      camera_hand="$(arg camera_hand)">
   </xacro:franka_robot>
 </robot>
