Commit message: Add minimic joit | Remap joint_states

File: robots/common/franka_arm.ros2_control.xacro (robot description, xacro)
@@ -25,5 +25,5 @@
           </xacro:if>
         </hardware>
-      <xacro:macro name="configure_joint" params="joint_name initial_position">
+      <xacro:macro name="configure_joint" params="joint_name initial_position:=^|0.0 mimic_joint:=^|''">
         <joint name="${joint_name}">
           <!--
@@ -37,9 +37,15 @@
           <command_interface name="position"/>
           <state_interface name="position">
-            <param name="initial_value">${initial_position}</param>
+            <xacro:if value="${mimic_joint == ''}">
+              <param name="initial_value">${initial_position}</param>
+            </xacro:if>
           </state_interface>
           <state_interface name="velocity"/>
             <param name="initial_value">0.0</param>
           <state_interface name="effort"/>
+          <xacro:if value="${mimic_joint != ''}">
+            <param name="mimic">${mimic_joint}</param>
+            <param name="multiplier">1</param>
+          </xacro:if>
         </joint>
       </xacro:macro>
@@ -53,4 +59,5 @@
       <xacro:if value="${gazebo and hand}">
         <xacro:configure_joint joint_name="${arm_id}_finger_joint1" initial_position="0.0" />
+        <xacro:configure_joint joint_name="${arm_id}_finger_joint2" mimic_joint="${arm_id}_finger_joint1"/>
       </xacro:if>
     </ros2_control>
@@ -59,4 +66,7 @@
         <plugin filename="franka_ign_ros2_control-system" name="ign_ros2_control::IgnitionROS2ControlPlugin">
           <parameters>$(find franka_gazebo_bringup)/config/franka_gazebo_controllers.yaml</parameters>
+          <ros>
+            <remapping>/joint_states:=/franka/joint_states</remapping>
+          </ros>
         </plugin>
       </gazebo>

Commit message: Remap simulation topics to mach real hardware

File: robots/common/franka_arm.ros2_control.xacro (robot description, xacro)
@@ -25,5 +25,5 @@
           </xacro:if>
         </hardware>
-      <xacro:macro name="configure_joint" params="joint_name initial_position">
+      <xacro:macro name="configure_joint" params="joint_name initial_position:=^|0.0 mimic_joint:=^|''">
         <joint name="${joint_name}">
           <!--
@@ -37,9 +37,15 @@
           <command_interface name="position"/>
           <state_interface name="position">
-            <param name="initial_value">${initial_position}</param>
+            <xacro:if value="${mimic_joint == ''}">
+              <param name="initial_value">${initial_position}</param>
+            </xacro:if>
           </state_interface>
           <state_interface name="velocity"/>
             <param name="initial_value">0.0</param>
           <state_interface name="effort"/>
+          <xacro:if value="${mimic_joint != ''}">
+            <param name="mimic">${mimic_joint}</param>
+            <param name="multiplier">1</param>
+          </xacro:if>
         </joint>
       </xacro:macro>
@@ -53,4 +59,5 @@
       <xacro:if value="${gazebo and hand}">
         <xacro:configure_joint joint_name="${arm_id}_finger_joint1" initial_position="0.0" />
+        <xacro:configure_joint joint_name="${arm_id}_finger_joint2" mimic_joint="${arm_id}_finger_joint1"/>
       </xacro:if>
     </ros2_control>
@@ -58,5 +65,15 @@
       <gazebo>
         <plugin filename="franka_ign_ros2_control-system" name="ign_ros2_control::IgnitionROS2ControlPlugin">
+<<<<<<< Updated upstream
           <parameters>$(find franka_gazebo_bringup)/config/franka_gazebo_controllers.yaml</parameters>
+=======
+          <parameters>${franka_controllers_params}</parameters>
+          <ros>
+            <remapping>/joint_states:=/franka/joint_states</remapping>
+            <remapping>/gripper_action_controller/gripper_cmd/_action/feedback:=/franka_gripper_node/gripper_action/_action/feedback</remapping>
+            <remapping>/gripper_action_controller/gripper_cmd/_action/status:=/franka_gripper_node/gripper_action/_action/status</remapping>
+            <remapping>/gripper_action_controller/transition_event:=/franka_gripper_node/transition_event</remapping>
+          </ros>
+>>>>>>> Stashed changes
         </plugin>
       </gazebo>

Commit message: Fix unresolved merge

File: robots/common/franka_arm.ros2_control.xacro (robot description, xacro)
@@ -25,5 +25,5 @@
           </xacro:if>
         </hardware>
-      <xacro:macro name="configure_joint" params="joint_name initial_position:=^|0.0 mimic_joint:=^|''">
+      <xacro:macro name="configure_joint" params="joint_name initial_position'">
         <joint name="${joint_name}">
           <!--
@@ -37,15 +37,9 @@
           <command_interface name="position"/>
           <state_interface name="position">
-            <xacro:if value="${mimic_joint == ''}">
               <param name="initial_value">${initial_position}</param>
-            </xacro:if>
           </state_interface>
           <state_interface name="velocity"/>
             <param name="initial_value">0.0</param>
           <state_interface name="effort"/>
-          <xacro:if value="${mimic_joint != ''}">
-            <param name="mimic">${mimic_joint}</param>
-            <param name="multiplier">1</param>
-          </xacro:if>
         </joint>
       </xacro:macro>
@@ -65,9 +59,6 @@
       <gazebo>
         <plugin filename="franka_ign_ros2_control-system" name="ign_ros2_control::IgnitionROS2ControlPlugin">
-<<<<<<< Updated upstream
           <parameters>$(find franka_gazebo_bringup)/config/franka_gazebo_controllers.yaml</parameters>
-=======
-          <parameters>${franka_controllers_params}</parameters>
-          <ros>
+           <ros>
             <remapping>/joint_states:=/franka/joint_states</remapping>
             <remapping>/gripper_action_controller/gripper_cmd/_action/feedback:=/franka_gripper_node/gripper_action/_action/feedback</remapping>
@@ -75,5 +66,4 @@
             <remapping>/gripper_action_controller/transition_event:=/franka_gripper_node/transition_event</remapping>
           </ros>
->>>>>>> Stashed changes
         </plugin>
       </gazebo>

Commit message: Fix leftovers form the merge

File: robots/common/franka_arm.ros2_control.xacro (robot description, xacro)
@@ -25,5 +25,5 @@
           </xacro:if>
         </hardware>
-      <xacro:macro name="configure_joint" params="joint_name initial_position'">
+      <xacro:macro name="configure_joint" params="joint_name initial_position">
         <joint name="${joint_name}">
           <!--
@@ -37,5 +37,5 @@
           <command_interface name="position"/>
           <state_interface name="position">
-              <param name="initial_value">${initial_position}</param>
+            <param name="initial_value">${initial_position}</param>
           </state_interface>
           <state_interface name="velocity"/>
@@ -53,5 +53,4 @@
       <xacro:if value="${gazebo and hand}">
         <xacro:configure_joint joint_name="${arm_id}_finger_joint1" initial_position="0.0" />
-        <xacro:configure_joint joint_name="${arm_id}_finger_joint2" mimic_joint="${arm_id}_finger_joint1"/>
       </xacro:if>
     </ros2_control>

Commit message: Add mimic joint (#16)
* Add minimic joit | Remap joint_states

* Remove topci remapping

File: robots/common/franka_arm.ros2_control.xacro (robot description, xacro)
@@ -35,5 +35,5 @@
           </xacro:if>
         </hardware>
-      <xacro:macro name="configure_joint" params="joint_name initial_position">
+      <xacro:macro name="configure_joint" params="joint_name initial_position:=^|0.0 mimic_joint:=^|''">
         <joint name="${joint_name}">
           <!--
@@ -50,9 +50,15 @@
           <!-- State Interfaces -->
           <state_interface name="position">
-            <param name="initial_value">${initial_position}</param>
+            <xacro:if value="${mimic_joint == ''}">
+              <param name="initial_value">${initial_position}</param>
+            </xacro:if>
           </state_interface>
           <state_interface name="velocity"/>
             <param name="initial_value">0.0</param>
           <state_interface name="effort"/>
+          <xacro:if value="${mimic_joint != ''}">
+            <param name="mimic">${mimic_joint}</param>
+            <param name="multiplier">1</param>
+          </xacro:if>
         </joint>
       </xacro:macro>
@@ -66,4 +72,5 @@
       <xacro:if value="${gazebo and hand}">
         <xacro:configure_joint joint_name="${arm_id}_finger_joint1" initial_position="0.0" />
+        <xacro:configure_joint joint_name="${arm_id}_finger_joint2" mimic_joint="${arm_id}_finger_joint1"/>
       </xacro:if>
     </ros2_control>
