Commit message: Add option to lock finger joints

File: end_effectors/common/franka_hand.xacro (robot description, xacro)
@@ -2,5 +2,5 @@
 <robot xmlns:xacro="http://www.ros.org/wiki/xacro" name="hand">
   <!-- safety_distance: Minimum safety distance in [m] by which the collision volumes are expanded and which is enforced during robot motions -->
-  <xacro:macro name="franka_hand" params="connected_to:='' arm_id ee_id ee_inertials rpy:='0 0 0' xyz:='0 0 0' tcp_xyz:='0 0 0.1034' tcp_rpy:='0 0 0' safety_distance:=0 gazebo:=false description_pkg:=franka_description with_sc:=false">
+  <xacro:macro name="franka_hand" params="connected_to:='' arm_id ee_id ee_inertials rpy:='0 0 0' xyz:='0 0 0' tcp_xyz:='0 0 0.1034' tcp_rpy:='0 0 0' safety_distance:=0 gazebo:=false description_pkg:=franka_description with_sc:=false lock_finger_joints:=false">
     <xacro:unless value="${connected_to == ''}">
       <joint name="${arm_id}_hand_joint" type="fixed">
@@ -100,5 +100,11 @@
       </xacro:if>
     </link>
-    <joint name="${arm_id}_finger_joint1" type="prismatic">
+    <xacro:if value="${lock_finger_joints}">
+      <xacro:property name="finger_joint_type" value="fixed" />
+    </xacro:if>
+    <xacro:unless value="${lock_finger_joints}">
+      <xacro:property name="finger_joint_type" value="prismatic" />
+    </xacro:unless>
+    <joint name="${arm_id}_finger_joint1" type="${finger_joint_type}">
       <parent link="${arm_id}_hand" />
       <child link="${arm_id}_leftfinger" />
@@ -108,5 +114,5 @@
       <dynamics damping="0.3" />
     </joint>
-    <joint name="${arm_id}_finger_joint2" type="prismatic">
+    <joint name="${arm_id}_finger_joint2" type="${finger_joint_type}">
       <parent link="${arm_id}_hand" />
       <child link="${arm_id}_rightfinger" />

File: end_effectors/franka_hand/franka_hand.urdf.xacro (robot description, xacro)
@@ -15,5 +15,6 @@
                      gazebo="$(arg gazebo)"
                      description_pkg="$(arg description_pkg)"
-                     with_sc="$(arg with_sc)">
+                     with_sc="$(arg with_sc)"
+                     lock_finger_joints="$(arg lock_finger_joints)">
    </xacro:franka_hand>
 </robot>

File: end_effectors/franka_hand/franka_hand_arguments.xacro (robot description, xacro)
@@ -25,3 +25,5 @@
   <!-- Should fake sensors be used? -->
   <xacro:arg name="description_pkg" default="franka_description" />
+  <!-- Should finger joints be locked? -->
+  <xacro:arg name="lock_finger_joints" default="false" />
 </robot>

File: robots/common/franka_robot.xacro (robot description, xacro)
@@ -56,4 +56,5 @@
         description_pkg="$(arg description_pkg)"
         with_sc="${with_sc}"
+        lock_finger_joints="$(arg lock_finger_joints)"
       />
     </xacro:if>
